File: PCB/avrwatch_v2/avrwatch_v2.kicad_sch (KiCad schematic)
At the start: 9 parts, among them J1 ICP, SW1 SW_Push, SW2 SW_Push, U1 ATmega328P-AU, U2 KCSA02-105, Y1 ABS07-120-32.768KHZ-T

Commit message: needs battery fixing
Parts:
- added P1: ~, QuorumPrecision:CR2032-120591, symbol QuorumPrecision:CR2032-120591
Connections:
- net GND: now also P1.2 (NEG)
- net VCC: now also P1.1 (POS)
